Commit message: fix standoffs

File: eddiebot_description/urdf/stacks/camera_stand.urdf.xacro (robot description, xacro)
@@ -93,6 +93,6 @@
         </inertial>
     </link>
-    <eddiebot_standoff_30cm parent="${parent}" number="0" x_loc="-0.140" y_loc="-0.084" z_loc="0.15715"/>
-    <eddiebot_standoff_30cm parent="${parent}" number="1" x_loc="-0.140" y_loc="0.084" z_loc="0.15715"/>
+    <xacro:eddiebot_standoff_30cm parent="${parent}" number="0" x_loc="-0.140" y_loc="-0.084" z_loc="0.15715"/>
+    <xacro:eddiebot_standoff_30cm parent="${parent}" number="1" x_loc="-0.140" y_loc="0.084" z_loc="0.15715"/>
   </xacro:macro>
 </robot>

File: eddiebot_description/urdf/stacks/circle_stack.urdf.xacro (robot description, xacro)
@@ -65,8 +65,8 @@
       </collision>
     </link>
-    <eddiebot_standoff_5in parent="${parent}" number="0" x_loc="0.0776402" y_loc="0.1314196" z_loc="0.06825"/>
-    <eddiebot_standoff_5in parent="${parent}" number="1" x_loc="0.0776402" y_loc="-0.1314196" z_loc="0.06825"/>
-    <eddiebot_standoff_5in parent="${parent}" number="2" x_loc="-0.0776402" y_loc="-0.1314196" z_loc="0.06825"/>
-    <eddiebot_standoff_5in parent="${parent}" number="3" x_loc="-0.0776402" y_loc="0.1314196" z_loc="0.06825"/>
+    <xacro:eddiebot_standoff_5in parent="${parent}" number="0" x_loc="0.0776402" y_loc="0.1314196" z_loc="0.06825"/>
+    <xacro:eddiebot_standoff_5in parent="${parent}" number="1" x_loc="0.0776402" y_loc="-0.1314196" z_loc="0.06825"/>
+    <xacro:eddiebot_standoff_5in parent="${parent}" number="2" x_loc="-0.0776402" y_loc="-0.1314196" z_loc="0.06825"/>
+    <xacro:eddiebot_standoff_5in parent="${parent}" number="3" x_loc="-0.0776402" y_loc="0.1314196" z_loc="0.06825"/>
   </xacro:macro>
 </robot>

File: eddiebot_description/urdf/stacks/create_base.urdf.xacro (robot description, xacro)
@@ -256,5 +256,5 @@
     </joint>
     <!-- This pretends to be in the center in order to aid in calculating degrees from multiple sensors on one fake laser scan -->
-    <!-- <joint name="ping_array_joint" type="fixed">
+    <joint name="ping_array_joint" type="fixed">
       <origin xyz="0 0 0.03695" rpy="0 0 0" />
       <parent link="base_link" />
@@ -274,6 +274,6 @@
           izz="0.0001" />
       </inertial>
-    </link> -->
-    <!-- <joint name="ir_array_joint" type="fixed">
+    </link>
+    <joint name="ir_array_joint" type="fixed">
       <origin xyz="0 0 0.03695" rpy="0 0 0" />
       <parent link="base_link" />
@@ -293,5 +293,5 @@
           izz="0.0001" />
       </inertial>
-    </link> -->
+    </link>
   </xacro:macro>
 </robot>
