Commit message: temp fix base_footprint inertia

File: eddiebot_description/urdf/stacks/create_base.urdf.xacro (robot description, xacro)
@@ -5,4 +5,9 @@
   <!-- <xacro:property name="base_x" value="0.33" /> -->
   <!-- <xacro:property name="base_y" value="0.33" /> -->
+  <xacro:macro name="box_inertial_matrix" params="m l w h">
+      <inertia ixx="${(m*(w*w+h*h))/12.0}" ixy = "0.0" ixz = "0.0"
+          iyy="${(m*(l*l+h*h))/12.0}" iyz = "0.0"
+          izz="${(m*(l*l+w*w))/12.0}" />
+  </xacro:macro>
   <xacro:macro name="create_base">
     <material name="Green">
@@ -17,17 +22,9 @@
     <!-- base_footprint is a fictitious link(frame) that is on the ground right below base_link origin, navigation stack depends on this frame -->
     <link name="base_footprint">
-      <visual>
-        <origin xyz="0 0 0" rpy="0 0 0" />
-        <geometry>
-          <box size="0.001 0.001 0.001" />
-        </geometry>
-        <material name="Green" />
-      </visual>
-      <collision>
-        <origin xyz="0 0 0.017" rpy="0 0 0" />
-        <geometry>
-          <box size="0.001 0.001 0.001" />
-        </geometry>
-      </collision>
+      <inertial>
+        <mass value="1" />
+        <origin xyz="0.0 0.0 0.0" />
+        <xacro:box_inertial_matrix m="1" h="1" l="1" w="1" />
+      </inertial>
     </link>
     <link name="base_link">

Commit message: add description launch

File: eddiebot_description/urdf/stacks/create_base.urdf.xacro (robot description, xacro)
@@ -20,4 +20,7 @@
       <color rgba="0.6 0.6 0.6 1"/>
     </material>
+    <material name="Black">
+        <color rgba="0.1 0.1 0.1 1"/>
+    </material>
     <!-- base_footprint is a fictitious link(frame) that is on the ground right below base_link origin, navigation stack depends on this frame -->
     <link name="base_footprint">
@@ -209,5 +212,5 @@
           <cylinder radius="0.0762" length = "0.03175"/>
         </geometry>
-        <material name ="black" />
+        <material name ="Black" />
       </visual>
       <collision>
@@ -238,5 +241,5 @@
           <cylinder radius="0.0762" length = "0.03175"/>
         </geometry>
-        <material name ="black" />
+        <material name ="Black" />
       </visual>
       <collision>

Commit message: clean up

File: eddiebot_description/urdf/stacks/create_base.urdf.xacro (robot description, xacro)
@@ -2,7 +2,4 @@
 <robot name="eddiebot_create_base" xmlns:xacro="http://ros.org/wiki/xacro">
   <xacro:property name="M_PI" value="3.1415926535897931" />
-  <!-- Macro for creating eddiebot base. -->
-  <!-- <xacro:property name="base_x" value="0.33" /> -->
-  <!-- <xacro:property name="base_y" value="0.33" /> -->
   <xacro:macro name="box_inertial_matrix" params="m l w h">
       <inertia ixx="${(m*(w*w+h*h))/12.0}" ixy = "0.0" ixz = "0.0"
@@ -11,8 +8,5 @@
   </xacro:macro>
   <xacro:macro name="create_base">
-    <material name="Green">
-      <color rgba="0.0 0.8 0.0 1.0"/>
-    </material>
-    <material name ="veryDarkGrey">
+    <material name ="dark_gray">
       <color rgba=".2 .2 .2 1"/>
     </material>
@@ -20,5 +14,5 @@
       <color rgba="0.6 0.6 0.6 1"/>
     </material>
-    <material name="Black">
+    <material name="black">
         <color rgba="0.1 0.1 0.1 1"/>
     </material>
@@ -43,5 +37,5 @@
           <cylinder length="0.0095" radius="0.2245"/>
         </geometry>
-        <material name ="veryDarkGrey" />
+        <material name ="dark_gray" />
       </visual>
       <collision>
@@ -52,93 +46,4 @@
       </collision>
     </link>
-    <link name="battery_box">
-      <inertial>
-        <mass value="0.001" />
-        <origin xyz="0 0 0" />
-        <inertia ixx="0.0001" ixy="0.0" ixz="0.0"
-          iyy="0.0001" iyz="0.0"
-          izz="0.0001" />
-      </inertial>
-      <visual>
-        <origin xyz="0 0 0" rpy="0 0 0" />
-        <geometry>
-          <box size="0.1778 0.3366 0.0762" />
-        </geometry>
-        <material name ="veryDarkGrey" />
-      </visual>
-      <collision>
-        <origin xyz="0 0 0" rpy="0 0 0" />
-        <geometry>
-          <box size="0.1778 0.3366 0.0762" />
-        </geometry>
-      </collision>
-    </link>
-    <joint name="battery_box_joint" type="fixed">
-      <origin xyz="0 0 -0.04285" rpy="0 0 0" />
-      <parent link="base_link" />
-      <child link="battery_box" />
-    </joint>
-    <link name="front_caster">
-      <inertial>
-        <mass value="0.001" />
-        <origin xyz="0 0 0" />
-        <inertia ixx="0.0001" ixy="0.0" ixz="0.0"
-          iyy="0.0001" iyz="0.0"
-          izz="0.0001" />
-      </inertial>
-      <visual>
-        <!-- <geometry>
-          <cylinder length="0.061" radius="0.05"/>
-        </geometry>
-        <origin rpy="${M_PI/2} 0 0" xyz="0 0 -0.05"/> -->
-        <origin xyz="0 0 0" rpy="-1.5707 0 1.5707" />
-        <geometry>
-          <mesh filename="package://eddiebot_description/meshes/28971-Caster-Wheel-Kit-v1.0.stl"/>
-        </geometry>
-        <material name ="light_grey">
-          <color rgba="0.6 0.6 0.6 1"/>
-        </material>
-      </visual>
-      <collision>
-        <geometry>
-          <cylinder length="0.061" radius="0.05"/>
-        </geometry>
-        <origin rpy="${M_PI/2} 0 0" xyz="0 0 -0.05"/>
-      </collision>
-    </link>
-    <joint name="front_caster_joint" type="fixed">
-      <origin xyz="0.18745 0 -0.00475" rpy="0 0 0" />
-      <parent link="base_link" />
-      <child link="front_caster" />
-    </joint>
-    <link name="rear_caster">
-      <inertial>
-        <mass value="0.001" />
-        <origin xyz="0 0 0" />
-        <inertia ixx="0.0001" ixy="0.0" ixz="0.0"
-          iyy="0.0001" iyz="0.0"
-          izz="0.0001" />
-      </inertial>
-      <visual>
-        <origin xyz="0 0 0" rpy="-1.5707 0 1.5707" />
-        <geometry>
-          <mesh filename="package://eddiebot_description/meshes/28971-Caster-Wheel-Kit-v1.0.stl"/>
-        </geometry>
-        <material name ="light_grey">
-          <color rgba="0.6 0.6 0.6 1"/>
-        </material>
-      </visual>
-      <collision>
-        <geometry>
-          <cylinder length="0.061" radius="0.05"/>
-        </geometry>
-        <origin rpy="${M_PI/2} 0 0" xyz="0 0 -0.05"/>
-      </collision>
-    </link>
-    <joint name="rear_caster_joint" type="fixed">
-      <origin xyz="-0.18745 0 -0.00475" rpy="0 0 0" />
-      <parent link="base_link" />
-      <child link="rear_caster" />
-    </joint>
     <joint name="base_footprint_joint" type="fixed">
       <origin xyz="0 0 0.10125" rpy="0 0 0" />
@@ -146,4 +51,93 @@
       <child link="base_link" />
     </joint>
+    <link name="battery_box">
+      <inertial>
+        <mass value="0.001" />
+        <origin xyz="0 0 0" />
+        <inertia ixx="0.0001" ixy="0.0" ixz="0.0"
+          iyy="0.0001" iyz="0.0"
+          izz="0.0001" />
+      </inertial>
+      <visual>
+        <origin xyz="0 0 0" rpy="0 0 0" />
+        <geometry>
+          <box size="0.1778 0.3366 0.0762" />
+        </geometry>
+        <material name ="dark_gray" />
+      </visual>
+      <collision>
+        <origin xyz="0 0 0" rpy="0 0 0" />
+        <geometry>
+          <box size="0.1778 0.3366 0.0762" />
+        </geometry>
+      </collision>
+    </link>
+    <joint name="battery_box_joint" type="fixed">
+      <origin xyz="0 0 -0.04285" rpy="0 0 0" />
+      <parent link="base_link" />
+      <child link="battery_box" />
+    </joint>
+    <link name="front_caster">
+      <inertial>
+        <mass value="0.001" />
+        <origin xyz="0 0 0" />
+        <inertia ixx="0.0001" ixy="0.0" ixz="0.0"
+          iyy="0.0001" iyz="0.0"
+          izz="0.0001" />
+      </inertial>
+      <visual>
+        <!-- <geometry>
+          <cylinder length="0.061" radius="0.05"/>
+        </geometry>
+        <origin rpy="${M_PI/2} 0 0" xyz="0 0 -0.05"/> -->
+        <origin xyz="0 0 0" rpy="-1.5707 0 1.5707" />
+        <geometry>
+          <mesh filename="package://eddiebot_description/meshes/28971-Caster-Wheel-Kit-v1.0.stl"/>
+        </geometry>
+        <material name ="light_grey">
+          <color rgba="0.6 0.6 0.6 1"/>
+        </material>
+      </visual>
+      <collision>
+        <geometry>
+          <cylinder length="0.061" radius="0.05"/>
+        </geometry>
+        <origin rpy="${M_PI/2} 0 0" xyz="0 0 -0.05"/>
+      </collision>
+    </link>
+    <joint name="front_caster_joint" type="fixed">
+      <origin xyz="0.18745 0 -0.00475" rpy="0 0 0" />
+      <parent link="base_link" />
+      <child link="front_caster" />
+    </joint>
+    <link name="rear_caster">
+      <inertial>
+        <mass value="0.001" />
+        <origin xyz="0 0 0" />
+        <inertia ixx="0.0001" ixy="0.0" ixz="0.0"
+          iyy="0.0001" iyz="0.0"
+          izz="0.0001" />
+      </inertial>
+      <visual>
+        <origin xyz="0 0 0" rpy="-1.5707 0 1.5707" />
+        <geometry>
+          <mesh filename="package://eddiebot_description/meshes/28971-Caster-Wheel-Kit-v1.0.stl"/>
+        </geometry>
+        <material name ="light_grey">
+          <color rgba="0.6 0.6 0.6 1"/>
+        </material>
+      </visual>
+      <collision>
+        <geometry>
+          <cylinder length="0.061" radius="0.05"/>
+        </geometry>
+        <origin rpy="${M_PI/2} 0 0" xyz="0 0 -0.05"/>
+      </collision>
+    </link>
+    <joint name="rear_caster_joint" type="fixed">
+      <origin xyz="-0.18745 0 -0.00475" rpy="0 0 0" />
+      <parent link="base_link" />
+      <child link="rear_caster" />
+    </joint>
     <link name="left_axle_link">
       <inertial>
@@ -212,5 +206,5 @@
           <cylinder radius="0.0762" length = "0.03175"/>
         </geometry>
-        <material name ="Black" />
+        <material name ="black" />
       </visual>
       <collision>
@@ -241,5 +235,5 @@
           <cylinder radius="0.0762" length = "0.03175"/>
         </geometry>
-        <material name ="Black" />
+        <material name ="black" />
       </visual>
       <collision>
@@ -258,4 +252,18 @@
       <axis xyz="0 1 0"/>
     </joint>
+    <link name="ping_sensor_array">
+      <visual>
+        <geometry>
+          <box size="0.0174 0.06 0.0644" />
+        </geometry>
+      </visual>
+      <inertial>
+        <mass value="0.001" />
+        <origin xyz="0 0 0" />
+        <inertia ixx="0.0001" ixy="0.0" ixz="0.0"
+          iyy="0.0001" iyz="0.0"
+          izz="0.0001" />
+      </inertial>
+    </link>
     <!-- This pretends to be in the center in order to aid in calculating degrees from multiple sensors on one fake laser scan -->
     <joint name="ping_array_joint" type="fixed">
@@ -264,5 +272,5 @@
       <child link="ping_sensor_array" />
     </joint>
-    <link name="ping_sensor_array">
+    <link name="ir_sensor_array">
       <visual>
         <geometry>
@@ -283,18 +291,4 @@
       <child link="ir_sensor_array" />
     </joint>
-    <link name="ir_sensor_array">
-      <visual>
-        <geometry>
-          <box size="0.0174 0.06 0.0644" />
-        </geometry>
-      </visual>
-      <inertial>
-        <mass value="0.001" />
-        <origin xyz="0 0 0" />
-        <inertia ixx="0.0001" ixy="0.0" ixz="0.0"
-          iyy="0.0001" iyz="0.0"
-          izz="0.0001" />
-      </inertial>
-    </link>
   </xacro:macro>
 </robot>
