Commit message: clean up

File: eddiebot_description/robots/eddie_kinect_v1/eddiebot.urdf.xacro (robot description, xacro)
@@ -14,3 +14,10 @@
   <xacro:camera_stand parent="plate_0_link"/>
   <xacro:sensor_kinect parent="camera_mount_link"/>
+  <!-- Listening on /model/$name/cmd_vel for velocity commands to move the robot -->
+  <gazebo>
+    <plugin
+      filename="gz-sim-velocity-control-system"
+      name="gz::sim::systems::VelocityControl">
+    </plugin>
+  </gazebo>
 </robot>

File: eddiebot_description/robots/eddiebot.urdf (robot description, URDF)
Before this commit: robot eddiebot, 24 links, 23 joints
Joints:
- joint right_wheel_joint: axis  -> 0 1 0; type revolute -> fixed

Commit message: eddiebot_description: use xacro properties

File: eddiebot_description/robots/eddie_kinect_v1/eddiebot.urdf.xacro (robot description, xacro)
@@ -1,13 +1,9 @@
 <?xml version="1.0"?>
 <robot name="eddiebot" xmlns:xacro="http://ros.org/wiki/xacro">
-  <!-- From $(find turtlebot_description)/urdf/common_properties.urdf.xacro -->
-  <!-- It is required by asus_xtion_pro.urdf.xacro (primesense carmine)-->
-  <xacro:property name="M_PI" value="3.1415926535897931" />
-  <!-- eddiebot base -->
   <xacro:include filename="$(find eddiebot_description)/urdf/stacks/create_base.urdf.xacro"/>
   <xacro:include filename="$(find eddiebot_description)/urdf/stacks/circle_stack.urdf.xacro"/>
   <xacro:include filename="$(find eddiebot_description)/urdf/stacks/camera_stand.urdf.xacro"/>
-  <!-- Kinect Sensor -->
   <xacro:include filename="$(find eddiebot_description)/urdf/sensors/kinect_v1.urdf.xacro"/>
+  <!-- eddiebot -->
   <xacro:create_base/>
   <xacro:circle_stack parent="base_link"/>

File: eddiebot_description/robots/eddiebot.urdf (robot description, URDF)
Before this commit: robot eddiebot, 24 links, 23 joints
Links:
- removed link ir_sensor_array
- removed link ping_sensor_array
- link base_footprint: mass 1 -> 2
- link battery_box: mass 0.001 -> 1
- link front_caster: mass 0.001 -> 0.8
- link left_axle_link: mass 0.01 -> 0.001
- link left_wheel_link: mass 0.01 -> 0.2
- link rear_caster: mass 0.001 -> 0.8; geometry collision sphere radius=0.05; visual mesh filename=package://eddiebot_description/meshes/28971-Caster-Wheel-Ki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
- link right_axle_link: mass 0.01 -> 0.001
- link right_wheel_link: mass 0.01 -> 0.2
Joints:
- removed joint ir_array_joint
- removed joint ping_array_joint
- joint front_caster_joint: type fixed -> continuous
- joint left_axle_joint: origin xyz=0 0.171475 0.0178 rpy=0 0 0 -> xyz=0 0.171475 0.017 rpy=0 0 0
- joint left_wheel_joint: type fixed -> continuous
- joint rear_caster_joint: type fixed -> continuous
- joint right_axle_joint: origin xyz=0 -0.171475 0.0178 rpy=0 0 0 -> xyz=0 -0.171475 0.017 rpy=0 0 0
- joint right_wheel_joint: type fixed -> continuous

File: eddiebot_description/urdf/stacks/camera_stand.urdf.xacro (robot description, xacro)
@@ -2,6 +2,4 @@
 <robot name="eddiebot_kinect_stand" xmlns:xacro="http://ros.org/wiki/xacro">
   <!-- Macro for creating eddiebot camera stand. -->
-  <!-- <xacro:property name="base_x" value="0.33" /> -->
-  <!-- <xacro:property name="base_y" value="0.33" /> -->
   <!-- Actually, the standoff is 30.48cm (12 inch)-->
   <xacro:macro name="eddiebot_standoff_30cm" params="parent number x_loc y_loc z_loc">
@@ -37,33 +35,4 @@
   </xacro:macro>
   <xacro:macro name="camera_stand" params="parent">
-    <!-- <joint name="plate_1_joint" type="fixed">
-      <origin xyz="0 0 0.1365" rpy="0 0 0" />
-      <parent link="${parent}"/>
-      <child link="plate_1_link" />
-    </joint>
-    <link name="plate_1_link">
-      <inertial>
-        <mass value="0.01" />
-        <origin xyz="0 0 0" />
-        <inertia ixx="0.01" ixy="0.0" ixz="0.0"
-          iyy="0.01" iyz="0.0"
-          izz="0.01" />
-      </inertial>
-      <visual>
-        <origin xyz=" 0 0 0 " rpy="0 0 0" />
-        <geometry>
-          <cylinder length="0.0095" radius="0.2245"/>
-        </geometry>
-        <material name ="veryDarkGrey">
-          <color rgba=".2 .2 .2 1"/>
-        </material>
-      </visual>
-      <collision>
-        <origin xyz="0.0 0.0 0.0" rpy="0 0 0" />
-        <geometry>
-          <cylinder length="0.0095" radius="0.2245"/>
-        </geometry>
-      </collision>
-    </link> -->
     <!-- Camera mount -->
     <joint name="camera_mount_joint" type="fixed">

File: eddiebot_description/urdf/stacks/circle_stack.urdf.xacro (robot description, xacro)
@@ -2,6 +2,4 @@
 <robot name="eddiebot_hardware" xmlns:xacro="http://ros.org/wiki/xacro">
   <!-- Macro for creating eddiebot circle stack. -->
-  <!-- <xacro:property name="base_x" value="0.33" /> -->
-  <!-- <xacro:property name="base_y" value="0.33" /> -->
   <xacro:macro name="eddiebot_standoff_5in" params="parent number x_loc y_loc z_loc">
     <joint name="standoff_5in_${number}_joint" type="fixed">

File: eddiebot_description/urdf/stacks/create_base.urdf.xacro (robot description, xacro)
@@ -1,99 +1,80 @@
 <?xml version="1.0"?>
 <robot name="eddiebot_create_base" xmlns:xacro="http://ros.org/wiki/xacro">
-  <xacro:property name="M_PI" value="3.1415926535897931" />
-  <xacro:macro name="box_inertial_matrix" params="m l w h">
-      <inertia ixx="${(m*(w*w+h*h))/12.0}" ixy = "0.0" ixz = "0.0"
-          iyy="${(m*(l*l+h*h))/12.0}" iyz = "0.0"
-          izz="${(m*(l*l+w*w))/12.0}" />
-  </xacro:macro>
+  <xacro:include filename="$(find eddiebot_description)/urdf/common.urdf.xacro"/>
+  <!-- Define robot constants -->
+  <xacro:property name="base_length" value="0.0095"/>
+  <xacro:property name="base_radius" value="0.2245"/>
+  <xacro:property name="base_mass" value="2"/>
+  <xacro:property name="base_link_z_offset" value="0.10125"/>
+  <xacro:property name="battery_box_z_offset" value="-0.04285"/>
+  <xacro:property name="battery_box_width" value="0.3366"/>
+  <xacro:property name="caster_mass" value="0.5"/>
+  <xacro:property name="caster_radius" value="0.05"/>
+  <xacro:property name="caster_length" value="0.061"/>
+  <xacro:property name="caster_x_offset" value="0.18745"/>
+  <xacro:property name="caster_z_offset" value="-0.00475"/>
+  <xacro:property name="axle_radius" value="0.00635"/>
+  <xacro:property name="axle_length" value="0.00635"/>
+  <xacro:property name="axle_y_offset" value="0.171475"/>
+  <xacro:property name="axle_z_offset" value="0.017"/>
+  <xacro:property name="wheel_mass" value="0.8"/>
+  <xacro:property name="wheel_radius" value="0.0762"/>
+  <xacro:property name="wheel_width" value="0.03175"/>
+  <xacro:property name="wheel_y_offset" value="0.01905"/>
   <xacro:macro name="create_base">
-    <material name ="dark_gray">
-      <color rgba=".2 .2 .2 1"/>
-    </material>
-    <material name ="light_grey">
-      <color rgba="0.6 0.6 0.6 1"/>
-    </material>
-    <material name="black">
-        <color rgba="0.1 0.1 0.1 1"/>
-    </material>
     <!-- base_footprint is a fictitious link(frame) that is on the ground right below base_link origin, navigation stack depends on this frame -->
     <link name="base_footprint">
-      <inertial>
-        <mass value="1" />
-        <origin xyz="0.0 0.0 0.0" />
-        <xacro:box_inertial_matrix m="1" h="1" l="1" w="1" />
-      </inertial>
-    </link>
-    <link name="base_link">
-      <inertial>
-        <mass value="2" />
-        <origin xyz="0 0 0.0" />
-        <inertia ixx="0.01" ixy="0.0" ixz="0.0"
-          iyy="0.01" iyz="0.0" izz="0.5" />
-      </inertial>
-      <visual>
-        <origin xyz="0 0 0" rpy="0 0 0" />
-        <geometry>
-          <cylinder length="0.0095" radius="0.2245"/>
-        </geometry>
-        <material name ="dark_gray" />
-      </visual>
-      <collision>
-        <origin xyz="0 0 0" rpy="0 0 0" />
-        <geometry>
-          <cylinder length="0.0095" radius="0.2245"/>
-        </geometry>
-      </collision>
+      <xacro:inertial_cylinder mass="${base_mass}" length="${base_length}" radius="${base_radius}"/>
     </link>
     <joint name="base_footprint_joint" type="fixed">
-      <origin xyz="0 0 0.10125" rpy="0 0 0" />
+      <origin xyz="0 0 ${base_link_z_offset}" rpy="0 0 0" />
       <parent link="base_footprint"/>
       <child link="base_link" />
     </joint>
+    <link name="base_link">
+      <xacro:inertial_cylinder mass="${base_mass}" length="${base_length}" radius="${base_radius}"/>
+      <visual>
+        <origin xyz="0 0 0" rpy="0 0 0" />
+        <geometry>
+          <cylinder length="${base_length}" radius="${base_radius}"/>
+        </geometry>
+        <material name ="material_darkgray" />
+      </visual>
+      <collision>
+        <origin xyz="0 0 0" rpy="0 0 0" />
+        <geometry>
+          <cylinder length="${base_length}" radius="${base_radius}"/>
+        </geometry>
+      </collision>
+    </link>
     <link name="battery_box">
-      <inertial>
-        <mass value="0.001" />
-        <origin xyz="0 0 0" />
-        <inertia ixx="0.0001" ixy="0.0" ixz="0.0"
-          iyy="0.0001" iyz="0.0"
-          izz="0.0001" />
-      </inertial>
-      <visual>
-        <origin xyz="0 0 0" rpy="0 0 0" />
-        <geometry>
-          <box size="0.1778 0.3366 0.0762" />
-        </geometry>
-        <material name ="dark_gray" />
-      </visual>
-      <collision>
-        <origin xyz="0 0 0" rpy="0 0 0" />
-        <geometry>
-          <box size="0.1778 0.3366 0.0762" />
+      <xacro:inertial_cuboid mass="1" x="0.1778" y="${battery_box_width}" z="0.0762"/>
+      <visual>
+        <origin xyz="0 0 0" rpy="0 0 0" />
+        <geometry>
+          <box size="0.1778 ${battery_box_width} 0.0762" />
+        </geometry>
+        <material name ="material_darkgray" />
+      </visual>
+      <collision>
+        <origin xyz="0 0 0" rpy="0 0 0" />
+        <geometry>
+          <box size="0.1778 ${battery_box_width} 0.0762" />
         </geometry>
       </collision>
     </link>
     <joint name="battery_box_joint" type="fixed">
-      <origin xyz="0 0 -0.04285" rpy="0 0 0" />
+      <origin xyz="0 0 ${battery_box_z_offset}" rpy="0 0 0" />
       <parent link="base_link" />
       <child link="battery_box" />
     </joint>
     <link name="front_caster">
-      <inertial>
-        <mass value="0.001" />
-        <origin xyz="0 0 0" />
-        <inertia ixx="0.0001" ixy="0.0" ixz="0.0"
-          iyy="0.0001" iyz="0.0"
-          izz="0.0001" />
-      </inertial>
-      <visual>
-        <!-- <geometry>
-          <cylinder length="0.061" radius="0.05"/>
-        </geometry>
-        <origin rpy="${M_PI/2} 0 0" xyz="0 0 -0.05"/> -->
-        <origin xyz="0 0 0" rpy="-1.5707 0 1.5707" />
+      <xacro:inertial_cylinder mass="${caster_mass}" length="${caster_length}" radius="${caster_radius}" />
+      <visual>
+        <origin xyz="0 0 0" rpy="-${M_PI/2} 0 ${M_PI/2}" />
         <geometry>
           <mesh filename="package://eddiebot_description/meshes/28971-Caster-Wheel-Kit-v1.0.stl"/>
         </geometry>
-        <material name ="light_grey">
+        <material name ="material_lightgray">
           <color rgba="0.6 0.6 0.6 1"/>
         </material>
@@ -101,28 +82,22 @@
       <collision>
         <geometry>
-          <cylinder length="0.061" radius="0.05"/>
-        </geometry>
-        <origin rpy="${M_PI/2} 0 0" xyz="0 0 -0.05"/>
+          <cylinder length="${caster_length}" radius="${caster_radius}"/>
+        </geometry>
+        <origin rpy="${M_PI/2} 0 0" xyz="0 0 -${caster_radius}"/>
       </collision>
     </link>
     <joint name="front_caster_joint" type="fixed">
-      <origin xyz="0.18745 0 -0.00475" rpy="0 0 0" />
+      <origin xyz="${caster_x_offset} 0 ${caster_z_offset}" rpy="0 0 0" />
       <parent link="base_link" />
       <child link="front_caster" />
     </joint>
     <link name="rear_caster">
-      <inertial>
-        <mass value="0.001" />
-        <origin xyz="0 0 0" />
-        <inertia ixx="0.0001" ixy="0.0" ixz="0.0"
-          iyy="0.0001" iyz="0.0"
-          izz="0.0001" />
-      </inertial>
-      <visual>
-        <origin xyz="0 0 0" rpy="-1.5707 0 1.5707" />
+      <xacro:inertial_cylinder mass="${caster_mass}" length="${caster_length}" radius="${caster_radius}" />
+      <visual>
+        <origin xyz="0 0 0" rpy="-${M_PI/2} 0 ${M_PI/2}" />
         <geometry>
           <mesh filename="package://eddiebot_description/meshes/28971-Caster-Wheel-Kit-v1.0.stl"/>
         </geometry>
-        <material name ="light_grey">
+        <material name ="material_lightgray">
           <color rgba="0.6 0.6 0.6 1"/>
         </material>
@@ -130,37 +105,32 @@
       <collision>
         <geometry>
-          <cylinder length="0.061" radius="0.05"/>
-        </geometry>
-        <origin rpy="${M_PI/2} 0 0" xyz="0 0 -0.05"/>
+          <sphere radius="${caster_radius}"/>
+        </geometry>
+        <origin rpy="${M_PI/2} 0 0" xyz="0 0 -${caster_radius}"/>
       </collision>
     </link>
     <joint name="rear_caster_joint" type="fixed">
-      <origin xyz="-0.18745 0 -0.00475" rpy="0 0 0" />
+      <origin xyz="${-caster_x_offset} 0 ${caster_z_offset}" rpy="0 0 0" />
       <parent link="base_link" />
       <child link="rear_caster" />
     </joint>
     <link name="left_axle_link">
-      <inertial>
-        <origin xyz="0 0 0"/>
-        <mass value="0.01" />
-        <inertia ixx="0.001" ixy="0.0" ixz="0.0"
-          iyy="0.001" iyz="0.0" izz="0.001" />
-      </inertial>
-      <visual>
-        <origin xyz="0 0 0" rpy="0 1.5707 1.5707" />
-        <geometry>
-          <cylinder radius="0.00635" length = "0.00635"/>
-        </geometry>
-        <material name ="light_grey" />
-      </visual>
-      <collision>
-        <origin xyz="0 0 0" rpy="0 1.5707 1.5707" />
-        <geometry>
-          <cylinder radius="0.00635" length = "0.00635"/>
+      <xacro:inertial_dummy />
+      <visual>
+        <origin xyz="0 0 0" rpy="0 ${M_PI/2} ${M_PI/2}" />
+        <geometry>
+          <cylinder radius="${axle_radius}" length = "${axle_length}"/>
+        </geometry>
+        <material name ="material_lightgray" />
+      </visual>
+      <collision>
+        <origin xyz="0 0 0" rpy="0 ${M_PI/2} ${M_PI/2}" />
+        <geometry>
+          <cylinder radius="${axle_radius}" length = "${axle_length}"/>
         </geometry>
       </collision>
     </link>
     <joint name="left_axle_joint" type="fixed">
-      <origin xyz="0 0.171475 0.0178" rpy="0 0 0"/>
+      <origin xyz="0 ${axle_y_offset} ${axle_z_offset}" rpy="0 0 0"/>
       <parent link="battery_box"/>
       <child link="left_axle_link"/>
@@ -168,26 +138,21 @@
     </joint>
     <link name="right_axle_link">
-      <inertial>
-        <origin xyz="0 0 0"/>
-        <mass value="0.01" />
-        <inertia ixx="0.001" ixy="0.0" ixz="0.0"
-          iyy="0.001" iyz="0.0" izz="0.001" />
-      </inertial>
-      <visual>
-        <origin xyz="0 0 0" rpy="0 1.5707 1.5707" />
-        <geometry>
-          <cylinder radius="0.00635" length = "0.00635"/>
-        </geometry>
-        <material name ="light_grey" />
-      </visual>
-      <collision>
-        <origin xyz="0 0 0" rpy="0 1.5707 1.5707" />
-        <geometry>
-          <cylinder radius="0.00635" length = "0.00635"/>
+      <xacro:inertial_dummy />
+      <visual>
+        <origin xyz="0 0 0" rpy="0 ${M_PI/2} ${M_PI/2}" />
+        <geometry>
+          <cylinder radius="${axle_radius}" length = "${axle_length}"/>
+        </geometry>
+        <material name ="material_lightgray" />
+      </visual>
+      <collision>
+        <origin xyz="0 0 0" rpy="0 ${M_PI/2} ${M_PI/2}" />
+        <geometry>
+          <cylinder radius="${axle_radius}" length = "${axle_length}"/>
         </geometry>
       </collision>
     </link>
     <joint name="right_axle_joint" type="fixed">
-      <origin xyz="0 -0.171475 0.0178" rpy="0 0 0"/>
+      <origin xyz="0 ${-axle_y_offset} ${axle_z_offset}" rpy="0 0 0"/>
       <parent link="battery_box"/>
       <child link="right_axle_link"/>
@@ -195,28 +160,21 @@
     </joint>
     <link name="left_wheel_link">
-      <inertial>
-        <origin xyz="0 0 0"/>
-        <mass value="0.01" />
-        <inertia ixx="0.001" ixy="0.0" ixz="0.0"
-          iyy="0.001" iyz="0.0" izz="0.001" />
-      </inertial>
-      <visual>
-        <origin xyz="0 0 0" rpy="0 1.5707 1.5707" />
-        <geometry>
-          <cylinder radius="0.0762" length = "0.03175"/>
-        </geometry>
-        <material name ="black" />
-      </visual>
-      <collision>
-        <origin xyz="0 0 0" rpy="0 1.5707 1.5707" />
-        <geometry>
-          <cylinder radius="0.0762" length = "0.03175"/>
-        </geometry>
-      </collision>
-    </link>
-    <!-- Fixed because we never rotate it anyway, it is just for show -->
-    <!-- NOTE This may prevent gazebo from working with this model -->
-    <joint name="left_wheel_joint" type="fixed">
-      <origin xyz="0 0.01905 0" rpy="0 0 0"/>
+      <xacro:inertial_cylinder mass="${wheel_mass}" radius="${wheel_radius}" length="${wheel_width}" />
+      <visual>
+        <origin xyz="0 0 0" rpy="${M_PI/2} 0 0" />
+        <geometry>
+          <cylinder radius="${wheel_radius}" length = "${wheel_width}"/>
+        </geometry>
+        <material name ="material_black" />
+      </visual>
+      <collision>
+        <origin xyz="0 0 0" rpy="${M_PI/2} 0 0" />
+        <geometry>
+          <cylinder radius="${wheel_radius}" length = "${wheel_width}"/>
+        </geometry>
+      </collision>
+    </link>
+    <joint name="left_wheel_joint" type="continuous">
+      <origin xyz="0 ${wheel_y_offset} 0" rpy="0 0 0"/>
       <parent link="left_axle_link"/>
       <child link="left_wheel_link"/>
@@ -224,73 +182,39 @@
     </joint>
     <link name="right_wheel_link">
-      <inertial>
-        <origin xyz="0 0 0"/>
-        <mass value="0.01" />
-        <inertia ixx="0.001" ixy="0.0" ixz="0.0"
-          iyy="0.001" iyz="0.0" izz="0.001" />
-      </inertial>
-      <visual>
-        <origin xyz="0 0 0" rpy="0 1.5707 1.5707" />
-        <geometry>
-          <cylinder radius="0.0762" length = "0.03175"/>
-        </geometry>
-        <material name ="black" />
-      </visual>
-      <collision>
-        <origin xyz="0 0 0" rpy="0 1.5707 1.5707" />
-        <geometry>
-          <cylinder radius="0.0762" length = "0.03175"/>
-        </geometry>
-      </collision>
-    </link>
-    <!-- Fixed because we never rotate it anyway, it is just for show -->
-    <!-- NOTE This may prevent gazebo from working with this model -->
-    <joint name="right_wheel_joint" type="fixed">
-      <origin xyz="0 -0.01905 0" rpy="0 0 0"/>
+      <xacro:inertial_cylinder mass="${wheel_mass}" radius="${wheel_radius}" length="${wheel_width}" />
+      <visual>
+        <origin xyz="0 0 0" rpy="${M_PI/2} 0 0" />
+        <geometry>
+          <cylinder radius="${wheel_radius}" length = "${wheel_width}"/>
+        </geometry>
+        <material name ="material_black" />
+      </visual>
+      <collision>
+        <origin xyz="0 0 0" rpy="${M_PI/2} 0 0" />
+        <geometry>
+          <cylinder radius="${wheel_radius}" length = "${wheel_width}"/>
+        </geometry>
+      </collision>
+    </link>
+    <joint name="right_wheel_joint" type="continuous">
+      <origin xyz="0 -${wheel_y_offset} 0" rpy="0 0 0"/>
       <parent link="right_axle_link"/>
       <child link="right_wheel_link"/>
       <axis xyz="0 1 0"/>
     </joint>
-    <link name="ping_sensor_array">
-      <visual>
-        <geometry>
-          <box size="0.0174 0.06 0.0644" />
-        </geometry>
-        <material name ="light_grey" />
-      </visual>
-      <inertial>
-        <mass value="0.001" />
-        <origin xyz="0 0 0" />
-        <inertia ixx="0.0001" ixy="0.0" ixz="0.0"
-          iyy="0.0001" iyz="0.0"
-          izz="0.0001" />
-      </inertial>
-    </link>
-    <!-- This pretends to be in the center in order to aid in calculating degrees from multiple sensors on one fake laser scan -->
-    <joint name="ping_array_joint" type="fixed">
-      <origin xyz="0 0 0.03695" rpy="0 0 0" />
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
Commit message: eddiebot_description: move to diff-drive

File: eddiebot_description/robots/eddie_kinect_v1/eddiebot.urdf.xacro (robot description, xacro)
@@ -10,10 +10,3 @@
   <xacro:camera_stand parent="plate_0_link"/>
   <xacro:sensor_kinect parent="camera_mount_link"/>
-  <!-- Listening on /model/$name/cmd_vel for velocity commands to move the robot -->
-  <gazebo>
-    <plugin
-      filename="gz-sim-velocity-control-system"
-      name="gz::sim::systems::VelocityControl">
-    </plugin>
-  </gazebo>
 </robot>

File: eddiebot_description/urdf/stacks/create_base.urdf.xacro (robot description, xacro)
@@ -17,5 +17,5 @@
   <xacro:property name="axle_length" value="0.00635"/>
   <xacro:property name="axle_y_offset" value="0.171475"/>
-  <xacro:property name="axle_z_offset" value="0.017"/>
+  <xacro:property name="axle_z_offset" value="0.014"/>
   <xacro:property name="wheel_mass" value="0.8"/>
   <xacro:property name="wheel_radius" value="0.0762"/>
@@ -87,4 +87,12 @@
       </collision>
     </link>
+    <gazebo reference="front_caster">
+      <mu1 value="0.0"/>
+      <mu2 value="0.0"/>
+      <kp value="10000000.0"/>
+      <kd value="1.0"/>
+      <fdir1 value="1 0 0"/>
+      <turnGravityOff>false</turnGravityOff>
+    </gazebo>
     <joint name="front_caster_joint" type="fixed">
       <origin xyz="${caster_x_offset} 0 ${caster_z_offset}" rpy="0 0 0" />
@@ -110,4 +118,12 @@
       </collision>
     </link>
+    <gazebo reference="rear_caster">
+      <mu1 value="0.0"/>
+      <mu2 value="0.0"/>
+      <kp value="10000000.0"/>
+      <kd value="1.0"/>
+      <fdir1 value="1 0 0"/>
+      <turnGravityOff>false</turnGravityOff>
+    </gazebo>
     <joint name="rear_caster_joint" type="fixed">
       <origin xyz="${-caster_x_offset} 0 ${caster_z_offset}" rpy="0 0 0" />
