Commit message: kinect: clean up

File: eddiebot_description/urdf/sensors/rgbd_sensor.urdf.xacro (robot description, xacro)
@@ -1,4 +1,7 @@
 <?xml version="1.0"?>
 <robot name="rgbd_sensor" xmlns:xacro="http://ros.org/wiki/xacro">
+    <xacro:property name="rgbd_fov" value="${60.0*M_PI/180.0}"/>
+    <xacro:property name="rgbd_width" value="640"/>
+    <xacro:property name="rgbd_height" value="480"/>
   <!-- Microsoft Kinect for simulation -->
     <xacro:macro name="rgbd_sensor_sim">
@@ -11,8 +14,8 @@
             <sensor name="camera" type="rgbd_camera">
                 <camera>
-                    <horizontal_fov>${60.0*M_PI/180.0}</horizontal_fov>
+                    <horizontal_fov>${rgbd_fov}</horizontal_fov>
                     <image>
-                        <width>640</width>
-                        <height>480</height>
+                        <width>${rgbd_width}</width>
+                        <height>${rgbd_height}</height>
                         <format>RGB_INT8</format>
                     </image>
@@ -21,4 +24,10 @@
                         <far>12.0</far>
                     </clip>
+                    <depth_camera>
+                        <clip>
+                            <near>0.05</near>
+                            <far>12.0</far>
+                        </clip>
+                    </depth_camera>
                     <distortion>
                         <k1>0.0</k1>
@@ -31,8 +40,11 @@
                     <lens>
                         <intrinsics>
-                            <fx>554.25469</fx>
-                            <fy>554.25469</fy>
-                            <cx>320.5</cx>
-                            <cy>240.5</cy>
+                            <!-- fx = fy = width / ( 2 * tan (hfov / 2 ) ) -->
+                            <fx>${rgbd_width / 2 * (0.5769)}</fx>
+                            <fy>${rgbd_width / 2 * (0.5769)}</fy>
+                            <!-- cx = ( width + 1 ) / 2 -->
+                            <cx>${(rgbd_width + 1)/2}</cx>
+                            <!-- cy = ( height + 1 ) / 2 -->
+                            <cy>${(rgbd_height + 1)/2}</cy>
                             <s>0</s>
                         </intrinsics>
@@ -43,10 +55,4 @@
                         <stddev>0.007</stddev>
                     </noise>
-                    <depth_camera>
-                        <clip>
-                            <near>0.05</near>
-                            <far>12.0</far>
-                        </clip>
-                    </depth_camera>
                 </camera>
                 <always_on>1</always_on>
