Commit message: Add ultrasonic sensor simulation macro
This commit adds a macro for simulating an ultrasonic sensor in the robot description. The macro includes the necessary elements such as the link, joint, and gazebo sensor. The sensor parameters are set to simulate a GPU lidar sensor with specific properties for scan, range, and noise. This macro can be used to easily add ultrasonic sensor simulations to the robot model.

Changes:
- Added macro ultrasonic_sensor_sim for simulating an ultrasonic sensor
- Included necessary elements such as link, joint, and gazebo sensor
- Configured sensor parameters for GPU lidar simulation with specific properties for scan, range, and noise

File: eddiebot_description/urdf/sensors/ultrasonic_sensor.urdf.xacro (robot description, xacro)
@@ -1,6 +1,6 @@
 <?xml version="1.0"?>
 <robot name="ultrasonic_sensor" xmlns:xacro="http://ros.org/wiki/xacro">
-    <xacro:property name="length" value="0.06"/>
-    <xacro:property name="width" value="0.01" />
+    <xacro:property name="length" value="0.01"/>
+    <xacro:property name="width" value="0.06" />
     <xacro:property name="height" value="0.03" />
     <xacro:macro name="ultrasonic_sensor_sim" params="name parent topic x y z roll pitch yaw linkname jointname">

Commit message: add ultasonic_sensor rotations to the link instead of the joint to keep the ray on the desired direction

File: eddiebot_description/urdf/sensors/ultrasonic_sensor.urdf.xacro (robot description, xacro)
@@ -49,5 +49,5 @@
         </link>
         <joint name="${joint_name}_2" type="fixed">
-            <origin xyz="0 -0.0225 0.015" rpy="${M_PI/2} 0 ${M_PI/2}"/>
+            <origin xyz="0 -0.0225 0.015" rpy="0 0 0"/>
             <parent link="${link_name}_1"/>
             <child link="${link_name}_2"/>
@@ -55,5 +55,5 @@
         <link name="${link_name}_2">
             <visual>
-                <origin xyz="0 0 0" rpy="0 0 0"/>
+                <origin xyz="0 0 0" rpy="${M_PI/2} 0 ${M_PI/2}"/>
                 <geometry>
                     <mesh filename="package://eddiebot_description/meshes/sensors/ultrasonic_infrared/ULTRASONIC_INFRARED.STL" scale="0.001 0.0009 0.0006"/>
@@ -62,5 +62,5 @@
             </visual>
             <collision>
-                <origin xyz="0 0 0" rpy="0 0 0"/>
+                <origin xyz="0 0 0" rpy="${M_PI/2} 0 ${M_PI/2}"/>
                 <geometry>
                     <box size="0.01 0.04 0.03"/>
