Commit message: create ir_sensor descriptions

File: eddiebot_description/urdf/sensors/ir_sensor.urdf.xacro (robot description, xacro)
@@ -19,58 +19,4 @@
             3- gazebo sensor: add gpu_lidar sensor with specified topic.
         -->
-        <joint name="${joint_name}" type="fixed">
-            <origin xyz="${x} ${y} ${z}" rpy="${roll} ${pitch} ${yaw}"/>
-            <parent link="${parent}"/>
-            <child link="${link_name}"/>
-        </joint>
-        <link name="${link_name}">
-            <visual>
-                <origin xyz="0 0 0" rpy="0 0 0"/>
-                <geometry>
-                    <box size="0.01 0.04 0.03"/>
-                </geometry>
-            </visual>
-            <collision>
-                <origin xyz="0.0 0.0 0.0" rpy="0 0 0"/>
-                <geometry>
-                    <box size="0.01 0.04 0.03"/>
-                </geometry>
-            </collision>
-            <inertial>
-                <mass value="0.1" />
-                <origin xyz="0 0 0" />
-                <inertia ixx="0.003881243" ixy="0.0" ixz="0.0"
-                        iyy="0.000498940" iyz="0.0"
-                        izz="0.003879257" />
-            </inertial>
-        </link>
-        <gazebo reference="${link_name}">
-            <sensor name="${sensor_name}" type='gpu_lidar'>
-                <always_on>1</always_on>
-                <update_rate>5</update_rate>
-                <visualize>1</visualize>
-                <topic>${topic_name}</topic>
-                <ray>
-                    <scan>
-                        <horizontal>
-                            <samples>1</samples>
-                            <resolution>1</resolution>
-                            <min_angle>0</min_angle>
-                            <max_angle>0</max_angle>
-                        </horizontal>
-                    </scan>
-                    <range>
-                        <min>0.1</min>
-                        <max>0.8</max>
-                        <resolution>0.02</resolution>
-                    </range>
-                    <noise>
-                        <type>gaussian</type>
-                        <mean>0.1</mean>
-                        <stddev>0.005</stddev>
-                    </noise>
-                </ray>
-            </sensor>
-        </gazebo>
     </xacro:macro>
 </robot>

Commit message: add ir_sensor link, joint and gzebo sensor

File: eddiebot_description/urdf/sensors/ir_sensor.urdf.xacro (robot description, xacro)
@@ -19,4 +19,58 @@
             3- gazebo sensor: add gpu_lidar sensor with specified topic.
         -->
+        <joint name="${joint_name}" type="fixed">
+            <origin xyz="${x} ${y} ${z}" rpy="${roll} ${pitch} ${yaw}"/>
+            <parent link="${parent}"/>
+            <child link="${link_name}"/>
+        </joint>
+        <link name="${link_name}">
+            <visual>
+                <origin xyz="0 0 0" rpy="0 0 0"/>
+                <geometry>
+                    <box size="0.01 0.04 0.03"/>
+                </geometry>
+            </visual>
+            <collision>
+                <origin xyz="0.0 0.0 0.0" rpy="0 0 0"/>
+                <geometry>
+                    <box size="0.01 0.04 0.03"/>
+                </geometry>
+            </collision>
+            <inertial>
+                <mass value="0.1" />
+                <origin xyz="0 0 0" />
+                <inertia ixx="0.003881243" ixy="0.0" ixz="0.0"
+                        iyy="0.000498940" iyz="0.0"
+                        izz="0.003879257" />
+            </inertial>
+        </link>
+        <gazebo reference="${link_name}">
+            <sensor name="${sensor_name}" type='gpu_lidar'>
+                <always_on>1</always_on>
+                <update_rate>5</update_rate>
+                <visualize>1</visualize>
+                <topic>${topic_name}</topic>
+                <ray>
+                    <scan>
+                        <horizontal>
+                            <samples>1</samples>
+                            <resolution>1</resolution>
+                            <min_angle>0</min_angle>
+                            <max_angle>0</max_angle>
+                        </horizontal>
+                    </scan>
+                    <range>
+                        <min>0.1</min>
+                        <max>0.8</max>
+                        <resolution>0.02</resolution>
+                    </range>
+                    <noise>
+                        <type>gaussian</type>
+                        <mean>0.1</mean>
+                        <stddev>0.005</stddev>
+                    </noise>
+                </ray>
+            </sensor>
+        </gazebo>
     </xacro:macro>
 </robot>

Commit message: add three ir sensors

File: eddiebot_description/urdf/sensors/ir_sensor.urdf.xacro (robot description, xacro)
@@ -1,5 +1,5 @@
 <?xml version="1.0"?>
 <robot name="infrared_sensor" xmlns:xacro="http://ros.org/wiki/xacro">
-    <xacro:include filename="$(find eddiebot_description)/urdf/common.urdf.xacro"/>
+    <!-- <xacro:include filename="$(find eddiebot_description)/urdf/common.urdf.xacro"/> -->
     <!--
         params:
@@ -26,8 +26,9 @@
         <link name="${link_name}">
             <visual>
-                <origin xyz="0 0 0" rpy="0 0 0"/>
+                <origin xyz="0 0 0" rpy="${M_PI/2} 0 ${M_PI/2}"/>
                 <geometry>
-                    <box size="0.01 0.04 0.03"/>
+                    <mesh filename="package://eddiebot_description/meshes/sensors/ultrasonic/ULTRASONICSENSOR.STL" scale="0.001 0.0009 0.0006"/>
                 </geometry>
+                <material name ="sensor_blue" />
             </visual>
             <collision>

File: eddiebot_description/urdf/stacks/create_base.urdf.xacro (robot description, xacro)
@@ -2,4 +2,5 @@
 <robot name="eddiebot_create_base" xmlns:xacro="http://ros.org/wiki/xacro">
   <xacro:include filename="$(find eddiebot_description)/urdf/sensors/ultrasonic_sensor.urdf.xacro"/>
+  <xacro:include filename="$(find eddiebot_description)/urdf/sensors/ir_sensor.urdf.xacro"/>
   <!-- Define robot constants -->
   <xacro:property name="base_length" value="0.0095"/>
@@ -235,6 +236,10 @@
     </gazebo>
     <!-- create two instances of the ultrasonic sensor -->
-    <xacro:ultrasonic_sensor topic_name="ultrasonic1" sensor_name="usen1" link_name="ul1" joint_name='uj1' parent="base_link" x="0.205" y="0.05" z="0.015" roll="0" pitch="0" yaw="${M_PI/8}"/>
-    <xacro:ultrasonic_sensor topic_name="ultrasonic2" sensor_name="usen2" link_name="ul2" joint_name='uj2' parent="base_link" x="0.190" y="-0.09" z="0.015" roll="0" pitch="0" yaw="${-M_PI/8}"/>
+    <xacro:ultrasonic_sensor topic_name="ultrasonic1" sensor_name="usen1" link_name="ul1" joint_name='uj1' parent="base_link" x="0.202" y="0.058" z="0.015" roll="0" pitch="0" yaw="${M_PI/8}"/>
+    <xacro:ultrasonic_sensor topic_name="ultrasonic2" sensor_name="usen2" link_name="ul2" joint_name='uj2' parent="base_link" x="0.185" y="-0.110" z="0.015" roll="0" pitch="0" yaw="${-M_PI/8}"/>
+    <!-- create three instances of the infrared sensor -->
+    <xacro:infrared_sensor topic_name="infrared1" sensor_name="isen1" link_name="il1" joint_name='ij1' parent="base_link" x="0.123" y="-0.167" z="0.030" roll="0" pitch="0" yaw="${-M_PI/4}"/>
+    <xacro:infrared_sensor topic_name="infrared2" sensor_name="isen2" link_name="il2" joint_name='ij2' parent="base_link" x="0.210" y="-0.03" z="0.030" roll="0" pitch="0" yaw="0"/>
+    <xacro:infrared_sensor topic_name="infrared3" sensor_name="isen3" link_name="il3" joint_name='ij3' parent="base_link" x="0.160" y="0.135" z="0.030" roll="0" pitch="0" yaw="${M_PI/4}"/>
   </xacro:macro>
 </robot>

Commit message: edit sensor mesh name and fix IR sensors positions

File: eddiebot_description/urdf/sensors/ir_sensor.urdf.xacro (robot description, xacro)
@@ -28,5 +28,5 @@
                 <origin xyz="0 0 0" rpy="${M_PI/2} 0 ${M_PI/2}"/>
                 <geometry>
-                    <mesh filename="package://eddiebot_description/meshes/sensors/ultrasonic/ULTRASONICSENSOR.STL" scale="0.001 0.0009 0.0006"/>
+                    <mesh filename="package://eddiebot_description/meshes/sensors/ultrasonic_infrared/ULTRASONIC_INFRARED.STL" scale="0.001 0.0009 0.0006"/>
                 </geometry>
                 <material name ="sensor_blue" />

File: eddiebot_description/urdf/sensors/ultrasonic_sensor.urdf.xacro (robot description, xacro)
@@ -28,5 +28,5 @@
                 <origin xyz="0 0 0" rpy="${M_PI/2} 0 ${M_PI/2}"/>
                 <geometry>
-                    <mesh filename="package://eddiebot_description/meshes/sensors/ultrasonic/ULTRASONICSENSOR.STL" scale="0.001 0.0009 0.0006"/>
+                    <mesh filename="package://eddiebot_description/meshes/sensors/ultrasonic_infrared/ULTRASONIC_INFRARED.STL" scale="0.001 0.0009 0.0006"/>
                 </geometry>
                 <material name ="sensor_blue" />

File: eddiebot_description/urdf/stacks/create_base.urdf.xacro (robot description, xacro)
@@ -236,9 +236,9 @@
     </gazebo>
     <!-- create two instances of the ultrasonic sensor -->
-    <xacro:ultrasonic_sensor topic_name="ultrasonic1" sensor_name="usen1" link_name="ul1" joint_name='uj1' parent="base_link" x="0.202" y="0.058" z="0.015" roll="0" pitch="0" yaw="${M_PI/8}"/>
+    <xacro:ultrasonic_sensor topic_name="ultrasonic1" sensor_name="usen1" link_name="ul1" joint_name='uj1' parent="base_link" x="0.20" y="0.058" z="0.015" roll="0" pitch="0" yaw="${M_PI/8}"/>
     <xacro:ultrasonic_sensor topic_name="ultrasonic2" sensor_name="usen2" link_name="ul2" joint_name='uj2' parent="base_link" x="0.185" y="-0.110" z="0.015" roll="0" pitch="0" yaw="${-M_PI/8}"/>
     <!-- create three instances of the infrared sensor -->
     <xacro:infrared_sensor topic_name="infrared1" sensor_name="isen1" link_name="il1" joint_name='ij1' parent="base_link" x="0.123" y="-0.167" z="0.030" roll="0" pitch="0" yaw="${-M_PI/4}"/>
-    <xacro:infrared_sensor topic_name="infrared2" sensor_name="isen2" link_name="il2" joint_name='ij2' parent="base_link" x="0.210" y="-0.03" z="0.030" roll="0" pitch="0" yaw="0"/>
+    <xacro:infrared_sensor topic_name="infrared2" sensor_name="isen2" link_name="il2" joint_name='ij2' parent="base_link" x="0.210" y="-0.028" z="0.030" roll="0" pitch="0" yaw="0"/>
     <xacro:infrared_sensor topic_name="infrared3" sensor_name="isen3" link_name="il3" joint_name='ij3' parent="base_link" x="0.160" y="0.135" z="0.030" roll="0" pitch="0" yaw="${M_PI/4}"/>
   </xacro:macro>

Commit message: added a stand for ultrasonic sensor

File: eddiebot_description/urdf/sensors/ir_sensor.urdf.xacro (robot description, xacro)
@@ -28,4 +28,5 @@
                 <origin xyz="0 0 0" rpy="${M_PI/2} 0 ${M_PI/2}"/>
                 <geometry>
+                    <!-- use STL file defined for both IR and ULTRASONIC sensors -->
                     <mesh filename="package://eddiebot_description/meshes/sensors/ultrasonic_infrared/ULTRASONIC_INFRARED.STL" scale="0.001 0.0009 0.0006"/>
                 </geometry>

File: eddiebot_description/urdf/sensors/ultrasonic_sensor.urdf.xacro (robot description, xacro)
@@ -19,12 +19,39 @@
             3- gazebo sensor: add gpu_lidar sensor with specified topic
         -->
-        <joint name="${joint_name}" type="fixed">
+        <joint name="${joint_name}_1" type="fixed">
             <origin xyz="${x} ${y} ${z}" rpy="${roll} ${pitch} ${yaw}"/>
             <parent link="${parent}"/>
-            <child link="${link_name}"/>
+            <child link="${link_name}_1"/>
         </joint>
-        <link name="${link_name}">
+        <link name="${link_name}_1">
             <visual>
-                <origin xyz="0 0 0" rpy="${M_PI/2} 0 ${M_PI/2}"/>
+                <origin xyz="0 0 0" rpy="0 0 0"/>
+                <geometry>
+                    <box size="0.01 0.01 0.04"/>
+                </geometry>
+                <material name ="material_darkgray" />
+            </visual>
+            <collision>
+                <origin xyz="0.0 0.0 0.0" rpy="0 0 0"/>
+                <geometry>
+                    <box size="0.01 0.01 0.04"/>
+                </geometry>
+            </collision>
+            <inertial>
+                <mass value="0.1" />
+                <origin xyz="0 0 0" />
+                <inertia ixx="0.003881243" ixy="0.0" ixz="0.0"
+                        iyy="0.000498940" iyz="0.0"
+                        izz="0.003879257" />
+            </inertial>
+        </link>
+        <joint name="${joint_name}_2" type="fixed">
+            <origin xyz="0 0 0" rpy="0 0 0"/>
+            <parent link="${link_name}_1"/>
+            <child link="${link_name}_2"/>
+        </joint>
+        <link name="${link_name}_2">
+            <visual>
+                <origin xyz="0 -0.0225 0.015" rpy="${M_PI/2} 0 ${M_PI/2}"/>
                 <geometry>
                     <mesh filename="package://eddiebot_description/meshes/sensors/ultrasonic_infrared/ULTRASONIC_INFRARED.STL" scale="0.001 0.0009 0.0006"/>
@@ -33,5 +60,5 @@
             </visual>
             <collision>
-                <origin xyz="0.0 0.0 0.0" rpy="0 0 0"/>
+                <origin xyz="0 -0.0225 0.015" rpy="${M_PI/2} 0 ${M_PI/2}"/>
                 <geometry>
                     <box size="0.01 0.04 0.03"/>
@@ -46,5 +73,5 @@
             </inertial>
         </link>
-        <gazebo reference="${link_name}">
+        <gazebo reference="${link_name}_2">
             <sensor name="${sensor_name}" type='gpu_lidar'>
                 <always_on>1</always_on>

File: eddiebot_description/urdf/stacks/create_base.urdf.xacro (robot description, xacro)
@@ -236,10 +236,10 @@
     </gazebo>
     <!-- create two instances of the ultrasonic sensor -->
-    <xacro:ultrasonic_sensor topic_name="ultrasonic1" sensor_name="usen1" link_name="ul1" joint_name='uj1' parent="base_link" x="0.20" y="0.058" z="0.015" roll="0" pitch="0" yaw="${M_PI/8}"/>
-    <xacro:ultrasonic_sensor topic_name="ultrasonic2" sensor_name="usen2" link_name="ul2" joint_name='uj2' parent="base_link" x="0.185" y="-0.110" z="0.015" roll="0" pitch="0" yaw="${-M_PI/8}"/>
+    <xacro:ultrasonic_sensor topic_name="ultrasonic1" sensor_name="usen1" link_name="ul1" joint_name='uj1' parent="base_link" x="0.195" y="0.09" z="0.015" roll="0" pitch="0" yaw="${M_PI/8}"/>
+    <xacro:ultrasonic_sensor topic_name="ultrasonic2" sensor_name="usen2" link_name="ul2" joint_name='uj2' parent="base_link" x="0.195" y="-0.09" z="0.015" roll="0" pitch="0" yaw="${-M_PI/8}"/>
     <!-- create three instances of the infrared sensor -->
-    <xacro:infrared_sensor topic_name="infrared1" sensor_name="isen1" link_name="il1" joint_name='ij1' parent="base_link" x="0.123" y="-0.167" z="0.030" roll="0" pitch="0" yaw="${-M_PI/4}"/>
-    <xacro:infrared_sensor topic_name="infrared2" sensor_name="isen2" link_name="il2" joint_name='ij2' parent="base_link" x="0.210" y="-0.028" z="0.030" roll="0" pitch="0" yaw="0"/>
-    <xacro:infrared_sensor topic_name="infrared3" sensor_name="isen3" link_name="il3" joint_name='ij3' parent="base_link" x="0.160" y="0.135" z="0.030" roll="0" pitch="0" yaw="${M_PI/4}"/>
+    <xacro:infrared_sensor topic_name="infrared1" sensor_name="isen1" link_name="il1" joint_name='ij1' parent="base_link" x="0.123" y="-0.167" z="0.025" roll="0" pitch="0" yaw="${-M_PI/4}"/>
+    <xacro:infrared_sensor topic_name="infrared2" sensor_name="isen2" link_name="il2" joint_name='ij2' parent="base_link" x="0.210" y="-0.028" z="0.025" roll="0" pitch="0" yaw="0"/>
+    <xacro:infrared_sensor topic_name="infrared3" sensor_name="isen3" link_name="il3" joint_name='ij3' parent="base_link" x="0.160" y="0.135" z="0.025" roll="0" pitch="0" yaw="${M_PI/4}"/>
   </xacro:macro>
 </robot>

Commit message: added stand for IR sensor and fixed the positions

File: eddiebot_description/urdf/sensors/ir_sensor.urdf.xacro (robot description, xacro)
@@ -14,19 +14,47 @@
     <xacro:macro name="infrared_sensor" params="topic_name sensor_name link_name joint_name parent x y z roll pitch yaw">
         <!--
-            there are three main parts,
-            1- joint: to connect parent link and sensor link.
-            2- link: small cuboid to represent the sensor.
-            3- gazebo sensor: add gpu_lidar sensor with specified topic.
+            <- main parts ->
+                1- first joint: to connect parent link and sensor stand link
+                2- first link: sensor stand
+                3- second joint: connect sensor link to the stand link
+                4- second link: sensor (using sensor STL file)
+                5- gazebo sensor: add gpu_lidar sensor with specified topic
         -->
-        <joint name="${joint_name}" type="fixed">
+        <joint name="${joint_name}_1" type="fixed">
             <origin xyz="${x} ${y} ${z}" rpy="${roll} ${pitch} ${yaw}"/>
             <parent link="${parent}"/>
-            <child link="${link_name}"/>
+            <child link="${link_name}_1"/>
         </joint>
-        <link name="${link_name}">
+        <link name="${link_name}_1">
             <visual>
-                <origin xyz="0 0 0" rpy="${M_PI/2} 0 ${M_PI/2}"/>
+                <origin xyz="0 0 0" rpy="0 0 0"/>
                 <geometry>
-                    <!-- use STL file defined for both IR and ULTRASONIC sensors -->
+                    <box size="0.01 0.01 0.05"/>
+                </geometry>
+                <material name ="material_darkgray" />
+            </visual>
+            <collision>
+                <origin xyz="0.0 0.0 0.0" rpy="0 0 0"/>
+                <geometry>
+                    <box size="0.01 0.01 0.05"/>
+                </geometry>
+            </collision>
+            <inertial>
+                <mass value="0.1" />
+                <origin xyz="0 0 0" />
+                <inertia ixx="0.003881243" ixy="0.0" ixz="0.0"
+                        iyy="0.000498940" iyz="0.0"
+                        izz="0.003879257" />
+            </inertial>
+        </link>
+        <joint name="${joint_name}_2" type="fixed">
+            <origin xyz="0 0 0" rpy="0 0 0"/>
+            <parent link="${link_name}_1"/>
+            <child link="${link_name}_2"/>
+        </joint>
+        <link name="${link_name}_2">
+            <visual>
+                <origin xyz="0 -0.0225 0.02" rpy="${M_PI/2} 0 ${M_PI/2}"/>
+                <geometry>
                     <mesh filename="package://eddiebot_description/meshes/sensors/ultrasonic_infrared/ULTRASONIC_INFRARED.STL" scale="0.001 0.0009 0.0006"/>
                 </geometry>
@@ -34,5 +62,5 @@
             </visual>
             <collision>
-                <origin xyz="0.0 0.0 0.0" rpy="0 0 0"/>
+                <origin xyz="0 -0.0225 0.02" rpy="${M_PI/2} 0 ${M_PI/2}"/>
                 <geometry>
                     <box size="0.01 0.04 0.03"/>
@@ -47,5 +75,5 @@
             </inertial>
         </link>
-        <gazebo reference="${link_name}">
+        <gazebo reference="${link_name}_2">
             <sensor name="${sensor_name}" type='gpu_lidar'>
                 <always_on>1</always_on>

File: eddiebot_description/urdf/stacks/create_base.urdf.xacro (robot description, xacro)
@@ -239,7 +239,7 @@
     <xacro:ultrasonic_sensor topic_name="ultrasonic2" sensor_name="usen2" link_name="ul2" joint_name='uj2' parent="base_link" x="0.195" y="-0.09" z="0.015" roll="0" pitch="0" yaw="${-M_PI/8}"/>
     <!-- create three instances of the infrared sensor -->
-    <xacro:infrared_sensor topic_name="infrared1" sensor_name="isen1" link_name="il1" joint_name='ij1' parent="base_link" x="0.123" y="-0.167" z="0.025" roll="0" pitch="0" yaw="${-M_PI/4}"/>
-    <xacro:infrared_sensor topic_name="infrared2" sensor_name="isen2" link_name="il2" joint_name='ij2' parent="base_link" x="0.210" y="-0.028" z="0.025" roll="0" pitch="0" yaw="0"/>
-    <xacro:infrared_sensor topic_name="infrared3" sensor_name="isen3" link_name="il3" joint_name='ij3' parent="base_link" x="0.160" y="0.135" z="0.025" roll="0" pitch="0" yaw="${M_PI/4}"/>
+    <xacro:infrared_sensor topic_name="infrared1" sensor_name="isen1" link_name="il1" joint_name='ij1' parent="base_link" x="0.135" y="-0.155" z="0.025" roll="0" pitch="0" yaw="${-M_PI/4}"/>
+    <xacro:infrared_sensor topic_name="infrared2" sensor_name="isen2" link_name="il2" joint_name='ij2' parent="base_link" x="0.210" y="0.00" z="0.025" roll="0" pitch="0" yaw="0"/>
+    <xacro:infrared_sensor topic_name="infrared3" sensor_name="isen3" link_name="il3" joint_name='ij3' parent="base_link" x="0.135" y="0.155" z="0.025" roll="0" pitch="0" yaw="${M_PI/4}"/>
   </xacro:macro>
 </robot>

Commit message: add ir_sensor rotations to the joint instead of link

File: eddiebot_description/urdf/sensors/ir_sensor.urdf.xacro (robot description, xacro)
@@ -49,5 +49,5 @@
         </link>
         <joint name="${joint_name}_2" type="fixed">
-            <origin xyz="0 0 0" rpy="0 0 0"/>
+            <origin xyz="0 -0.0225 0.02" rpy="${M_PI/2} 0 ${M_PI/2}"/>
             <parent link="${link_name}_1"/>
             <child link="${link_name}_2"/>
@@ -55,5 +55,5 @@
         <link name="${link_name}_2">
             <visual>
-                <origin xyz="0 -0.0225 0.02" rpy="${M_PI/2} 0 ${M_PI/2}"/>
+                <origin xyz="0 0 0" rpy="0 0 0"/>
                 <geometry>
                     <mesh filename="package://eddiebot_description/meshes/sensors/ultrasonic_infrared/ULTRASONIC_INFRARED.STL" scale="0.001 0.0009 0.0006"/>
@@ -62,5 +62,5 @@
             </visual>
             <collision>
-                <origin xyz="0 -0.0225 0.02" rpy="${M_PI/2} 0 ${M_PI/2}"/>
+                <origin xyz="0 0 0" rpy="0 0 0"/>
                 <geometry>
                     <box size="0.01 0.04 0.03"/>
