Commit message: add rotations to the link instead of the joint to keep the ray on the desired direction

File: eddiebot_description/urdf/sensors/ir_sensor.urdf.xacro (robot description, xacro)
@@ -49,5 +49,5 @@
         </link>
         <joint name="${joint_name}_2" type="fixed">
-            <origin xyz="0 -0.0225 0.02" rpy="${M_PI/2} 0 ${M_PI/2}"/>
+            <origin xyz="0 -0.0225 0.02" rpy="0 0 0"/>
             <parent link="${link_name}_1"/>
             <child link="${link_name}_2"/>
@@ -55,5 +55,5 @@
         <link name="${link_name}_2">
             <visual>
-                <origin xyz="0 0 0" rpy="0 0 0"/>
+                <origin xyz="0 0 0" rpy="${M_PI/2} 0 ${M_PI/2}"/>
                 <geometry>
                     <mesh filename="package://eddiebot_description/meshes/sensors/ultrasonic_infrared/ULTRASONIC_INFRARED.STL" scale="0.001 0.0009 0.0006"/>

File: eddiebot_description/urdf/sensors/ultrasonic_sensor.urdf.xacro (robot description, xacro)
@@ -49,5 +49,5 @@
         </link>
         <joint name="${joint_name}_2" type="fixed">
-            <origin xyz="0 0 0" rpy="0 0 0"/>
+            <origin xyz="0 -0.0225 0.015" rpy="${M_PI/2} 0 ${M_PI/2}"/>
             <parent link="${link_name}_1"/>
             <child link="${link_name}_2"/>
@@ -55,5 +55,5 @@
         <link name="${link_name}_2">
             <visual>
-                <origin xyz="0 -0.0225 0.015" rpy="${M_PI/2} 0 ${M_PI/2}"/>
+                <origin xyz="0 0 0" rpy="0 0 0"/>
                 <geometry>
                     <mesh filename="package://eddiebot_description/meshes/sensors/ultrasonic_infrared/ULTRASONIC_INFRARED.STL" scale="0.001 0.0009 0.0006"/>
@@ -62,5 +62,5 @@
             </visual>
             <collision>
-                <origin xyz="0 -0.0225 0.015" rpy="${M_PI/2} 0 ${M_PI/2}"/>
+                <origin xyz="0 0 0" rpy="0 0 0"/>
                 <geometry>
                     <box size="0.01 0.04 0.03"/>

Commit message: added third joint and link to correct the ray direction

File: eddiebot_description/urdf/sensors/ir_sensor.urdf.xacro (robot description, xacro)
@@ -75,5 +75,11 @@
             </inertial>
         </link>
-        <gazebo reference="${link_name}_2">
+        <joint name="${joint_name}_3" type="fixed">
+            <origin xyz="0 0.025 0.02" rpy="0 0 0"/>
+            <parent link="${link_name}_2"/>
+            <child link="${link_name}_3"/>
+        </joint>
+        <link name="${link_name}_3"/>
+        <gazebo reference="${link_name}_3">
             <sensor name="${sensor_name}" type='gpu_lidar'>
                 <always_on>1</always_on>

Commit message: IR and Ultrasonic sensors placed

File: eddiebot_description/urdf/sensors/ir_sensor.urdf.xacro (robot description, xacro)
@@ -1,6 +1,5 @@
 <?xml version="1.0"?>
-<robot name="ultrasonic_ping_1" xmlns:xacro="http://ros.org/wiki/xacro">
-    <!-- <xacro:include filename="$(find eddiebot_description)/urdf/common.urdf.xacro"/> -->
-    <xacro:macro name="ultrasonic_ping" params="name x y z r p ya">
+<robot name="ir_ping" xmlns:xacro="http://ros.org/wiki/xacro">
+    <xacro:macro name="ir_ping" params="name x y z r p ya">
             <link name="${name}_link">
                 <xacro:inertial_cuboid mass="0.3" x="0.1778" y="0.18" z="0.0762" />
@@ -9,5 +8,5 @@
                     <origin xyz="0 0 0" rpy="0 0 0" />
                     <geometry>
-                        <box size="0.01 0.04 0.025" />
+                        <box size="0.01 0.02 0.04" />
                     </geometry>
                 </visual>
@@ -15,5 +14,5 @@
                   <origin xyz="0 0 0" rpy="0 0 0" />
                   <geometry>
-                    <box size="0.01 0.04 0.025" />
+                    <box size="0.01 0.02 0.04" />
                   </geometry>
                 </collision>

File: eddiebot_description/urdf/stacks/create_base.urdf.xacro (robot description, xacro)
@@ -3,4 +3,5 @@
   <xacro:include filename="$(find eddiebot_description)/urdf/common.urdf.xacro"/>
   <xacro:include filename="$(find eddiebot_description)/urdf/sensors/ultrasonic_sensor.urdf.xacro"/>
+  <xacro:include filename="$(find eddiebot_description)/urdf/sensors/ir_sensor.urdf.xacro"/>
   <!-- Define robot constants -->
   <xacro:property name="base_length" value="0.0095"/>
@@ -48,6 +49,9 @@
       </collision>
     </link>
-    <xacro:ultrasonic_ping name="ultra1" x="0.18" y="-0.05" z="0.0165" r="0" p="0" ya="-0.2" />
-    <xacro:ultrasonic_ping name="ultra2" x="0.18" y="0.05" z="0.0165" r="0" p="0" ya="0.2" />
+    <xacro:ultrasonic_ping name="ultra_r" x="0.18" y="-0.07" z="0.0165" r="0" p="0" ya="-0.2" />
+    <xacro:ultrasonic_ping name="ultra_l" x="0.18" y="0.07" z="0.0165" r="0" p="0" ya="0.2" />
+    <xacro:ir_ping name="ir_r" x="0.15" y="-0.12" z="0.025" r="0" p="0" ya="-0.6" />
+    <xacro:ir_ping name="ir_l" x="0.15" y="0.12" z="0.025" r="0" p="0" ya="0.6" />
+    <xacro:ir_ping name="ir_c" x="0.187" y="0" z="0.025" r="0" p="0" ya="0" />
     <link name="battery_box">
       <xacro:inertial_cuboid mass="1" x="0.1778" y="${battery_box_width}" z="0.0762"/>

Commit message: IR and Ultrasonic sensors placed

File: eddiebot_description/urdf/sensors/ir_sensor.urdf.xacro (robot description, xacro)
@@ -1,26 +1,39 @@
 <?xml version="1.0"?>
 <robot name="ir_ping" xmlns:xacro="http://ros.org/wiki/xacro">
+    <!-- in this file we have the desctibtion of IR sensor which uses light to
+    measure and recognize the distances such as measuring the distance which the
+    robot is away from the wall or trying not to hit walls or any other objects
+    we have 6 main parameters which will be passed when an instance is being created.
+    name which is the name of the ir sensor, x which is the distance on the axis of x which
+    the robot is away from the `base_link`, y and z are the same. r is the roll rotation,
+    p is the pitch rotation and ya is the yaw rotation-->
     <xacro:macro name="ir_ping" params="name x y z r p ya">
-            <link name="${name}_link">
-                <xacro:inertial_cuboid mass="0.3" x="0.1778" y="0.18" z="0.0762" />
-                <visual>
-                    <material name="material_darkgray" />
-                    <origin xyz="0 0 0" rpy="0 0 0" />
-                    <geometry>
-                        <box size="0.01 0.02 0.04" />
-                    </geometry>
-                </visual>
-                <collision>
-                  <origin xyz="0 0 0" rpy="0 0 0" />
-                  <geometry>
+        <!-- Link of the ir sensor. the difference between the ultrasonic sensor
+        is that this sensor is narrower than the physical form of ultrasonic sensors-->
+        <link name="${name}_link">
+            <xacro:inertial_cuboid mass="0.3" x="0.1778" y="0.18" z="0.0762" />
+            <visual>
+                <material name="material_darkgray" />
+                <origin xyz="0 0 0" rpy="0 0 0" />
+                <geometry>
                     <box size="0.01 0.02 0.04" />
-                  </geometry>
-                </collision>
-            </link>
-            <joint name="${name}_joint" type="fixed">
-              <origin xyz="${x} ${y} ${z}" rpy="${r} ${p} ${ya}" />
-              <parent link="base_link" />
-              <child link="${name}_link" />
-            </joint>
+                </geometry>
+            </visual>
+            <collision>
+              <origin xyz="0 0 0" rpy="0 0 0" />
+              <geometry>
+                <box size="0.01 0.02 0.04" />
+              </geometry>
+            </collision>
+        </link>
+        <!-- We need joint for describtion of our sensor which is obvious in the
+        follow -->
+        <joint name="${name}_joint" type="fixed">
+          <origin xyz="${x} ${y} ${z}" rpy="${r} ${p} ${ya}" />
+          <parent link="base_link" />
+          <child link="${name}_link" />
+        </joint>
+        <!-- here we describe the sensor. its name, sample rates, the topic it
+        poblishes the informations to, resolution and etc. -->
         <gazebo reference="${name}_link">
             <sensor name='${name}' type='gpu_lidar'>

File: eddiebot_description/urdf/sensors/ultrasonic_sensor.urdf.xacro (robot description, xacro)
@@ -1,27 +1,38 @@
 <?xml version="1.0"?>
 <robot name="ultrasonic_ping_1" xmlns:xacro="http://ros.org/wiki/xacro">
-    <!-- <xacro:include filename="$(find eddiebot_description)/urdf/common.urdf.xacro"/> -->
+    <!-- In this file we have the describtion of Ultrasonic sensor which uses
+    ultrasonic sound waves to measure the distance from objects around.
+    we have 6 main parameters which will be passed when an instance is being created.
+    name which is the name of the ir sensor, x which is the distance on the axis of x which
+    the robot is away from the `base_link`, y and z are the same. r is the roll rotation,
+    p is the pitch rotation and ya is the yaw rotation-->
     <xacro:macro name="ultrasonic_ping" params="name x y z r p ya">
-            <link name="${name}_link">
-                <xacro:inertial_cuboid mass="0.3" x="0.1778" y="0.18" z="0.0762" />
-                <visual>
-                    <material name="material_darkgray" />
-                    <origin xyz="0 0 0" rpy="0 0 0" />
-                    <geometry>
-                        <box size="0.01 0.04 0.025" />
-                    </geometry>
-                </visual>
-                <collision>
-                  <origin xyz="0 0 0" rpy="0 0 0" />
-                  <geometry>
+        <!-- link of the ultrasonic sensor. which has informations like sensor's visual
+        look and collision-->
+        <link name="${name}_link">
+            <xacro:inertial_cuboid mass="0.3" x="0.1778" y="0.18" z="0.0762" />
+            <visual>
+                <material name="material_darkgray" />
+                <origin xyz="0 0 0" rpy="0 0 0" />
+                <geometry>
                     <box size="0.01 0.04 0.025" />
-                  </geometry>
-                </collision>
-            </link>
-            <joint name="${name}_joint" type="fixed">
-              <origin xyz="${x} ${y} ${z}" rpy="${r} ${p} ${ya}" />
-              <parent link="base_link" />
-              <child link="${name}_link" />
-            </joint>
+                </geometry>
+            </visual>
+            <collision>
+              <origin xyz="0 0 0" rpy="0 0 0" />
+              <geometry>
+                <box size="0.01 0.04 0.025" />
+              </geometry>
+            </collision>
+        </link>
+        <!-- We need joint for describtion of our sensor which is obvious in the
+        follow -->
+        <joint name="${name}_joint" type="fixed">
+          <origin xyz="${x} ${y} ${z}" rpy="${r} ${p} ${ya}" />
+          <parent link="base_link" />
+          <child link="${name}_link" />
+        </joint>
+        <!-- here we describe the sensor. its name, sample rates, the topic it
+        poblishes the informations to, resolution and etc. -->
         <gazebo reference="${name}_link">
             <sensor name='${name}' type='gpu_lidar'>
