Commit message: add STL mesh for ultrasonic sensor

File: eddiebot_description/urdf/common.urdf.xacro (robot description, xacro)
@@ -55,4 +55,7 @@
     <color rgba="0.3 0.3 0.3 1"/>
   </material>
+  <material name="sensor_blue">
+    <color rgba="0.1 0.2 0.8 1"/>
+  </material>
   <material name="material_lightgray">
     <color rgba="0.5 0.5 0.5 1"/>

File: eddiebot_description/urdf/sensors/ir_sensor.urdf.xacro (robot description, xacro)
@@ -1,21 +1,21 @@
 <?xml version="1.0"?>
-<robot name="ultrasonic_sensor" xmlns:xacro="http://ros.org/wiki/xacro">
+<robot name="infrared_sensor" xmlns:xacro="http://ros.org/wiki/xacro">
     <xacro:include filename="$(find eddiebot_description)/urdf/common.urdf.xacro"/>
     <!--
         params:
-        1- topic name: name of the gazebo topic for ultrasonic sensor
-        2- sensor name: name of the sensor
-        3- link name: name of the link for ultrasonic sensor, since there are more than one
+        1: topic name: name of the gazebo topic for infrared sensor
+        2: sensor name: name of the sensor
+        3: link name: name of the link for infrared sensor, since there are more than one
             sensors, link name is set as an parameter to prevent the name consistency.
-        4- joint name: name of the joint, to prevent the name consistency same as the link name.
-        5- parent name: name of the paranet, to connect joints between parent and link_name
-        6,11- parameters for specifying the position of sensor on the base link.
+        4: joint name: name of the joint, to prevent the name consistency same as the link name.
+        5: parent name: name of the paranet, to connect joints between parent and link_name
+        6-11: parameters for specifying the position of sensor on the base link.
     -->
-    <xacro:macro name="ultrasonic_sensor" params="topic_name sensor_name link_name joint_name parent x y z roll pitch yaw">
+    <xacro:macro name="infrared_sensor" params="topic_name sensor_name link_name joint_name parent x y z roll pitch yaw">
         <!--
             there are three main parts,
-            1- joint: to connect parent link and sensor link
-            2- link: small cuboid to represent the sensor
-            3- gazebo sensor: add gpu_lidar sensor with specified topic
+            1- joint: to connect parent link and sensor link.
+            2- link: small cuboid to represent the sensor.
+            3- gazebo sensor: add gpu_lidar sensor with specified topic.
         -->
         <joint name="${joint_name}" type="fixed">
@@ -26,9 +26,8 @@
         <link name="${link_name}">
             <visual>
-                <origin xyz="0 0 0" rpy="${M_PI/2} 0 ${M_PI/2}"/>
+                <origin xyz="0 0 0" rpy="0 0 0"/>
                 <geometry>
-                    <mesh filename="package://eddiebot_description/meshes/sensors/ultrasonic/ULTRASONICSENSOR.STL" scale="0.001 0.0009 0.0006"/>
+                    <box size="0.01 0.04 0.03"/>
                 </geometry>
-                <material name ="sensor_blue" />
             </visual>
             <collision>
@@ -62,6 +61,6 @@
                     </scan>
                     <range>
-                        <min>0.08</min>
-                        <max>4</max>
+                        <min>0.1</min>
+                        <max>0.8</max>
                         <resolution>0.02</resolution>
                     </range>

File: eddiebot_description/urdf/stacks/create_base.urdf.xacro (robot description, xacro)
@@ -235,6 +235,6 @@
     </gazebo>
     <!-- create two instances of the ultrasonic sensor -->
-    <xacro:ultrasonic_sensor topic_name="ultrasonic1" sensor_name="usen1" link_name="ul1" joint_name='uj1' parent="base_link" x="0.205" y="0.07" z="0.015" roll="0" pitch="0" yaw="${M_PI/8}"/>
-    <xacro:ultrasonic_sensor topic_name="ultrasonic2" sensor_name="usen2" link_name="ul2" joint_name='uj2' parent="base_link" x="0.205" y="-0.07" z="0.015" roll="0" pitch="0" yaw="${-M_PI/8}"/>
+    <xacro:ultrasonic_sensor topic_name="ultrasonic1" sensor_name="usen1" link_name="ul1" joint_name='uj1' parent="base_link" x="0.205" y="0.05" z="0.015" roll="0" pitch="0" yaw="${M_PI/8}"/>
+    <xacro:ultrasonic_sensor topic_name="ultrasonic2" sensor_name="usen2" link_name="ul2" joint_name='uj2' parent="base_link" x="0.190" y="-0.09" z="0.015" roll="0" pitch="0" yaw="${-M_PI/8}"/>
   </xacro:macro>
 </robot>
