Commit message: add eddiebot_gazebo

File: eddiebot_description/robots/eddiebot.urdf (robot description, URDF)
Before this commit: robot eddiebot, 24 links, 23 joints
Joints:
- joint right_wheel_joint: axis 0 1 0 -> ; type fixed -> revolute

File: eddiebot_description/urdf/stacks/create_base.urdf.xacro (robot description, xacro)
@@ -257,4 +257,5 @@
           <box size="0.0174 0.06 0.0644" />
         </geometry>
+        <material name ="light_grey" />
       </visual>
       <inertial>
@@ -277,4 +278,5 @@
           <box size="0.0174 0.06 0.0644" />
         </geometry>
+        <material name ="black" />
       </visual>
       <inertial>

Commit message: nav: clean up

File: eddiebot_description/robots/eddiebot.urdf (robot description, URDF)
Before this commit: robot eddiebot, 22 links, 21 joints
Links:
- link base_footprint: mass 2 -> None
- link front_caster: mass 0.8 -> 0.5
- link left_wheel_link: mass 0.2 -> 0.8
- link rear_caster: mass 0.8 -> 0.5
- link right_wheel_link: mass 0.2 -> 0.8
Joints:
- joint front_caster_joint: type continuous -> fixed
- joint left_axle_joint: origin xyz=0 0.171475 0.017 rpy=0 0 0 -> xyz=0 0.171475 0.014 rpy=0 0 0
- joint rear_caster_joint: type continuous -> fixed
- joint right_axle_joint: origin xyz=0 -0.171475 0.017 rpy=0 0 0 -> xyz=0 -0.171475 0.014 rpy=0 0 0

Commit message: lab 10

File: eddiebot_description/robots/eddiebot.urdf (robot description, URDF)
Before this commit: robot eddiebot, 22 links, 21 joints
Links:
- link base_footprint: mass 2 -> None
- link front_caster: mass 0.8 -> 0.5
- link left_wheel_link: mass 0.2 -> 0.8
- link rear_caster: mass 0.8 -> 0.5
- link right_wheel_link: mass 0.2 -> 0.8
Joints:
- joint front_caster_joint: type continuous -> fixed
- joint left_axle_joint: origin xyz=0 0.171475 0.017 rpy=0 0 0 -> xyz=0 0.171475 0.014 rpy=0 0 0
- joint rear_caster_joint: type continuous -> fixed
- joint right_axle_joint: origin xyz=0 -0.171475 0.017 rpy=0 0 0 -> xyz=0 -0.171475 0.014 rpy=0 0 0

File: eddiebot_description/urdf/stacks/create_base.urdf.xacro (robot description, xacro)
@@ -2,4 +2,5 @@
 <robot name="eddiebot_create_base" xmlns:xacro="http://ros.org/wiki/xacro">
   <xacro:include filename="$(find eddiebot_description)/urdf/common.urdf.xacro"/>
+  <xacro:include filename="$(find eddiebot_description)/urdf/sensors/ultrasonic_sensor.urdf.xacro"/>
   <!-- Define robot constants -->
   <xacro:property name="base_length" value="0.0095"/>
@@ -47,4 +48,6 @@
       </collision>
     </link>
+    <xacro:ultrasonic_ping name="ultra1" x="0.18" y="-0.05" z="0.0165" r="0" p="0" ya="-0.2" />
+    <xacro:ultrasonic_ping name="ultra2" x="0.18" y="0.05" z="0.0165" r="0" p="0" ya="0.2" />
     <link name="battery_box">
       <xacro:inertial_cuboid mass="1" x="0.1778" y="${battery_box_width}" z="0.0762"/>
